File: pcb/sensorline.brd (EAGLE design)
At the start: 141 x 21.3 mm, 31 parts, among them X1 52745-1290

Commit message: a takie tam poprawki
Parts:
- added JP1, JP2: (no value), pinhead:1X03
- X1: value 52745-1290 -> FH12-14S-0.5SH; device con-molex:52745-1290 -> con-hirose:FH12-14S-0.5SH
- moved X1 6.84 mm to (85.1, 3.81)
Connections:
- new net N$21: JP1.1, X1.1
- new net N$22: JP2.1, X1.2
- net GND: now also JP1.3, JP2.3, X1.13; no longer X1.11
- net N$10: now also X1.8; no longer X1.6
- net N$12: now also X1.7; no longer X1.5
- net N$14: now also X1.6; no longer X1.4
- net N$16: now also X1.5; no longer X1.3
- net N$18: now also X1.4; no longer X1.2
- net N$2: now also X1.12; no longer X1.10
- net N$20: now also X1.3; no longer X1.1
- net N$4: now also X1.11; no longer X1.9
- net N$6: now also X1.10; no longer X1.8
- net N$8: now also X1.9; no longer X1.7
- net VCC: now also JP1.2, JP2.2, X1.14; no longer X1.12
Changed lines of the file:
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@@
 <?xml version="1.0" encoding="utf-8"?>
 <!DOCTYPE eagle SYSTEM "eagle.dtd">
-<eagle version="7.1.0">
+<eagle version="8.1.1">
 <drawing>
 <settings>
@@
 <element name="R8" library="rcl" package="R0402" value="10k" x="97.79" y="19.05"/>
 <element name="R9" library="rcl" package="R0402" value="330" x="86.36" y="13.97"/>
-<element name="X1" library="con-molex" package="52745-1290" value="52745-1290" x="78.74" y="1.27">
-<attribute name="OC_NEWARK" value="92M6383" x="78.74" y="1.27" size="1.778" layer="27" display="off"/>
-<attribute name="MPN" value="52745-1290" x="78.74" y="1.27" size="1.778" layer="27" display="off"/>
-<attribute name="MF" value="" x="78.74" y="1.27" size="1.778" layer="27" display="off"/>
-<attribute name="OC_FARNELL" value="unknown" x="78.74" y="1.27" size="1.778" layer="27" display="off"/>
+<element name="X1" library="con-hirose" package="FH12-14S-0.5SH" value="FH12-14S-0.5SH" x="85.09" y="3.81">
+<attribute name="MF" value="" x="85.09" y="3.81" size="1.778" layer="27" display="off"/>
+<attribute name="MPN" value="MC34827" x="85.09" y="3.81" size="1.778" layer="27" display="off"/>
+<attribute name="OC_FARNELL" value="1324544" x="85.09" y="3.81" size="1.778" layer="27" display="off"/>
+<attribute name="OC_NEWARK" value="41P0493" x="85.09" y="3.81" size="1.778" layer="27" display="off"/>
 </element>
+<element name="JP1" library="pinhead" package="1X03" value="" x="71.12" y="3.81"/>
+<element name="JP2" library="pinhead" package="1X03" value="" x="101.6" y="3.81"/>
 </elements>
 <signals>
@@
 <contactref element="CZ7" pad="KOLEKTOR"/>
 <contactref element="R3" pad="2"/>
-<contactref element="X1" pad="10"/>
-<wire x1="80.49" y1="3.77" x2="153.115" y2="17.42" width="0" layer="19" extent="1-1"/>
-<wire x1="47.64" y1="19.05" x2="80.49" y2="3.77" width="0" layer="19" extent="1-1"/>
+<contactref element="X1" pad="12"/>
+<wire x1="47.64" y1="19.05" x2="153.115" y2="17.42" width="0" layer="19" extent="1-1"/>
+<wire x1="87.34" y1="7.06" x2="47.64" y2="19.05" width="0" layer="19" extent="1-1"/>
 </signal>
 <signal name="GND">
@@
 <contactref element="CZ10" pad="EMITER"/>
 <contactref element="CZ10" pad="KATODA"/>
-<contactref element="X1" pad="11"/>
+<contactref element="X1" pad="13"/>
+<contactref element="JP1" pad="3"/>
+<contactref element="JP2" pad="3"/>
 <wire x1="149.145" y1="17.41" x2="153.115" y2="15.61" width="0" layer="19" extent="1-1"/>
 <wire x1="139.145" y1="15.61" x2="149.145" y2="17.41" width="0" layer="19" extent="1-1"/>
@@
 <wire x1="27.385" y1="15.61" x2="37.385" y2="17.41" width="0" layer="19" extent="1-1"/>
 <wire x1="23.415" y1="17.41" x2="27.385" y2="15.61" width="0" layer="19" extent="1-1"/>
-<wire x1="80.99" y1="3.77" x2="79.455" y2="15.61" width="0" layer="19" extent="1-1"/>
+<wire x1="87.84" y1="7.06" x2="27.385" y2="15.61" width="0" layer="19" extent="1-1"/>
+<wire x1="73.66" y1="3.81" x2="87.84" y2="7.06" width="0" layer="19" extent="1-1"/>
+<wire x1="104.14" y1="3.81" x2="73.66" y2="3.81" width="0" layer="19" extent="1-1"/>
 </signal>
 <signal name="VCC">
@@
 <contactref element="R19" pad="1"/>
 <contactref element="R20" pad="2"/>
-<contactref element="X1" pad="12"/>
+<contactref element="X1" pad="14"/>
+<contactref element="JP2" pad="2"/>
+<contactref element="JP1" pad="2"/>
 <wire x1="146.7" y1="13.97" x2="146.7" y2="19.05" width="0" layer="19" extent="1-1"/>
 <wire x1="132.73" y1="13.97" x2="146.7" y2="13.97" width="0" layer="19" extent="1-1"/>
@@
 <wire x1="87.01" y1="13.97" x2="97.14" y2="19.05" width="0" layer="19" extent="1-1"/>
 <wire x1="85.71" y1="19.05" x2="87.01" y2="13.97" width="0" layer="19" extent="1-1"/>
-<wire x1="81.49" y1="3.77" x2="87.01" y2="13.97" width="0" layer="19" extent="1-1"/>
 <wire x1="71.74" y1="19.05" x2="85.71" y2="19.05" width="0" layer="19" extent="1-1"/>
 <wire x1="71.77" y1="13.97" x2="71.74" y2="19.05" width="0" layer="19" extent="1-1"/>
@@
 <wire x1="19.67" y1="19.05" x2="33.64" y2="19.05" width="0" layer="19" extent="1-1"/>
 <wire x1="19.67" y1="13.97" x2="19.67" y2="19.05" width="0" layer="19" extent="1-1"/>
+<wire x1="88.34" y1="7.06" x2="19.67" y2="13.97" width="0" layer="19" extent="1-1"/>
+<wire x1="71.12" y1="3.81" x2="88.34" y2="7.06" width="0" layer="19" extent="1-1"/>
+<wire x1="101.6" y1="3.81" x2="71.12" y2="3.81" width="0" layer="19" extent="1-1"/>
 </signal>
 <signal name="N$3">
@@
 <contactref element="CZ1" pad="KOLEKTOR"/>
 <contactref element="R1" pad="2"/>
-<contactref element="X1" pad="9"/>
-<wire x1="79.99" y1="3.77" x2="139.145" y2="17.42" width="0" layer="19" extent="1-1"/>
-<wire x1="59.07" y1="19.05" x2="79.99" y2="3.77" width="0" layer="19" extent="1-1"/>
+<contactref element="X1" pad="11"/>
+<wire x1="59.07" y1="19.05" x2="139.145" y2="17.42" width="0" layer="19" extent="1-1"/>
+<wire x1="86.84" y1="7.06" x2="59.07" y2="19.05" width="0" layer="19" extent="1-1"/>
 </signal>
 <signal name="N$5">
@@
 <contactref element="CZ2" pad="KOLEKTOR"/>
 <contactref element="R4" pad="2"/>
-<contactref element="X1" pad="8"/>
-<wire x1="79.49" y1="3.77" x2="125.175" y2="17.42" width="0" layer="19" extent="1-1"/>
-<wire x1="34.94" y1="19.05" x2="79.49" y2="3.77" width="0" layer="19" extent="1-1"/>
+<contactref element="X1" pad="10"/>
+<wire x1="34.94" y1="19.05" x2="125.175" y2="17.42" width="0" layer="19" extent="1-1"/>
+<wire x1="86.34" y1="7.06" x2="34.94" y2="19.05" width="0" layer="19" extent="1-1"/>
 </signal>
 <signal name="N$7">
@@
 <contactref element="CZ3" pad="KOLEKTOR"/>
 <contactref element="R6" pad="2"/>
-<contactref element="X1" pad="7"/>
-<wire x1="78.99" y1="3.77" x2="109.935" y2="17.42" width="0" layer="19" extent="1-1"/>
-<wire x1="20.97" y1="19.05" x2="78.99" y2="3.77" width="0" layer="19" extent="1-1"/>
+<contactref element="X1" pad="9"/>
+<wire x1="85.84" y1="7.06" x2="109.935" y2="17.42" width="0" layer="19" extent="1-1"/>
+<wire x1="20.97" y1="19.05" x2="85.84" y2="7.06" width="0" layer="19" extent="1-1"/>
 </signal>
 <signal name="N$9">
@@
 <contactref element="CZ4" pad="KOLEKTOR"/>
 <contactref element="R8" pad="2"/>
-<contactref element="X1" pad="6"/>
+<contactref element="X1" pad="8"/>
 <wire x1="94.695" y1="17.42" x2="98.44" y2="19.05" width="0" layer="19" extent="1-1"/>
-<wire x1="78.49" y1="3.77" x2="94.695" y2="17.42" width="0" layer="19" extent="1-1"/>
+<wire x1="85.34" y1="7.06" x2="94.695" y2="17.42" width="0" layer="19" extent="1-1"/>
 </signal>
 <signal name="N$11">
@@
 <contactref element="CZ5" pad="KOLEKTOR"/>
 <contactref element="R10" pad="2"/>
-<contactref element="X1" pad="5"/>
+<contactref element="X1" pad="7"/>
 <wire x1="79.455" y1="17.42" x2="87.01" y2="19.05" width="0" layer="19" extent="1-1"/>
-<wire x1="77.99" y1="3.77" x2="79.455" y2="17.42" width="0" layer="19" extent="1-1"/>
+<wire x1="84.84" y1="7.06" x2="79.455" y2="17.42" width="0" layer="19" extent="1-1"/>
 </signal>
 <signal name="N$13">
@@
 <contactref element="CZ6" pad="KOLEKTOR"/>
 <contactref element="R12" pad="2"/>
-<contactref element="X1" pad="4"/>
-<wire x1="77.49" y1="3.77" x2="145.4" y2="19.05" width="0" layer="19" extent="1-1"/>
-<wire x1="65.485" y1="17.42" x2="77.49" y2="3.77" width="0" layer="19" extent="1-1"/>
+<contactref element="X1" pad="6"/>
+<wire x1="65.485" y1="17.42" x2="145.4" y2="19.05" width="0" layer="19" extent="1-1"/>
+<wire x1="84.34" y1="7.06" x2="65.485" y2="17.42" width="0" layer="19" extent="1-1"/>
 </signal>
 <signal name="N$15">
@@
 <contactref element="CZ8" pad="KOLEKTOR"/>
 <contactref element="R14" pad="2"/>
-<contactref element="X1" pad="3"/>
-<wire x1="76.99" y1="3.77" x2="114.95" y2="19.05" width="0" layer="19" extent="1-1"/>
-<wire x1="52.785" y1="17.42" x2="76.99" y2="3.77" width="0" layer="19" extent="1-1"/>
+<contactref element="X1" pad="5"/>
+<wire x1="52.785" y1="17.42" x2="114.95" y2="19.05" width="0" layer="19" extent="1-1"/>
+<wire x1="83.84" y1="7.06" x2="52.785" y2="17.42" width="0" layer="19" extent="1-1"/>
 </signal>
 <signal name="N$17">
@@
 <contactref element="CZ9" pad="KOLEKTOR"/>
 <contactref element="R17" pad="2"/>
-<contactref element="X1" pad="2"/>
-<wire x1="41.355" y1="17.42" x2="76.49" y2="3.77" width="0" layer="19" extent="1-1"/>
+<contactref element="X1" pad="4"/>
 <wire x1="34.94" y1="13.97" x2="41.355" y2="17.42" width="0" layer="19" extent="1-1"/>
+<wire x1="83.34" y1="7.06" x2="34.94" y2="13.97" width="0" layer="19" extent="1-1"/>
 </signal>
 <signal name="N$19">
@@
 <contactref element="CZ10" pad="KOLEKTOR"/>
 <contactref element="R19" pad="2"/>
+<contactref element="X1" pad="3"/>
+<wire x1="27.385" y1="17.42" x2="73.04" y2="19.05" width="0" layer="19" extent="1-1"/>
+<wire x1="82.84" y1="7.06" x2="27.385" y2="17.42" width="0" layer="19" extent="1-1"/>
+</signal>
+<signal name="N$21">
+<contactref element="JP1" pad="1"/>
 <contactref element="X1" pad="1"/>
-<wire x1="75.99" y1="3.77" x2="73.04" y2="19.05" width="0" layer="19" extent="1-1"/>
-<wire x1="27.385" y1="17.42" x2="73.04" y2="19.05" width="0" layer="19" extent="1-1"/>
+<wire x1="68.58" y1="3.81" x2="81.84" y2="7.06" width="0" layer="19" extent="1-1"/>
+</signal>
+<signal name="N$22">
+<contactref element="JP2" pad="1"/>
+<contactref element="X1" pad="2"/>
+<wire x1="99.06" y1="3.81" x2="82.34" y2="7.06" width="0" layer="19" extent="1-1"/>
 </signal>
 </signals>

Commit message: o już niewiele
Parts:
- removed CZ10, CZ9: KTIR0711S, KTIR0711S:TOP
- removed R1, R10, R12, R14, R17, R19, R3, R4, R6, R8: 10k, rcl:R0402
- removed R11, R13, R15, R16, R18, R2, R20, R5, R7, R9: 330, rcl:R0402
- added CZ0, CZ19: KTIR0711S, KTIR0711S:TOP
- added RN1, RN2, RN3, RN4, RN5, RN6: CTS742C083, resistor-net:CTS742C083
- moved CZ1 176.1 mm to (-38.0, -2.30), flipped to the bottom, turned to 180 degrees
- moved CZ2 151.7 mm to (-27.6, 0.24), flipped to the bottom, turned to 180 degrees
- moved CZ7 127.5 mm to (24.6, 0.24), flipped to the bottom, turned to 180 degrees
- moved CZ3 126.5 mm to (-17.6, 1.51), flipped to the bottom, turned to 180 degrees
- moved CZ4 101.5 mm to (-7.63, 1.51), flipped to the bottom, turned to 180 degrees
- moved JP2 97.0 mm to (4.62, 6.91)
- moved X1 86.8 mm to (-1.42, -3.85)
- moved JP1 79.0 mm to (-7.81, 6.91)
- moved CZ5 74.4 mm to (4.63, 1.51), flipped to the bottom, turned to 180 degrees
- moved CZ6 51.1 mm to (14.6, 1.51), flipped to the bottom, turned to 180 degrees
- moved CZ8 25.0 mm to (34.3, -2.30), flipped to the bottom, turned to 180 degrees
Connections:
- net GND: now also CZ0.EMITER, CZ0.KATODA, CZ19.EMITER, CZ19.KATODA; no longer CZ10.EMITER, CZ10.KATODA, CZ9.EMITER, CZ9.KATODA
- net N$1: now also CZ0.ANODA, RN1.2; no longer CZ7.ANODA, R16.1
- net N$10: now also RN5.1, X1.7; no longer R8.2, X1.8
- net N$11: now also RN2.1; no longer R11.1
- net N$12: now also RN5.2, X1.8; no longer R10.2, X1.7
- net N$13: now also RN2.4; no longer R13.1
- net N$14: now also RN5.3, X1.9; no longer R12.2, X1.6
- net N$15: now also CZ7.ANODA, RN2.3; no longer CZ8.ANODA, R15.1
- net N$16: now also CZ7.KOLEKTOR, RN5.4, X1.10; no longer CZ8.KOLEKTOR, R14.2, X1.5
- net N$17: now also CZ8.ANODA, RN3.1; no longer CZ9.ANODA, R18.1
- net N$18: now also CZ8.KOLEKTOR, RN6.2, X1.11; no longer CZ9.KOLEKTOR, R17.2, X1.4
- net N$19: now also CZ19.ANODA, RN3.2; no longer CZ10.ANODA, R20.1
- net N$2: now also CZ0.KOLEKTOR, RN4.1, X1.3; no longer CZ7.KOLEKTOR, R3.2, X1.12
- net N$20: now also CZ19.KOLEKTOR, RN6.1, X1.12; no longer CZ10.KOLEKTOR, R19.2, X1.3
- net N$3: now also RN1.1; no longer R2.1
- net N$4: now also RN4.2, X1.4; no longer R1.2, X1.11
- net N$5: now also RN1.4; no longer R5.1
- net N$6: now also RN4.3, X1.5; no longer R4.2, X1.10
- net N$7: now also RN1.3; no longer R7.1
- net N$8: now also RN4.4, X1.6; no longer R6.2, X1.9
- net N$9: now also RN2.2; no longer R9.1
- net VCC: now also RN1.5, RN1.6, RN1.7, RN1.8, RN2.5, RN2.6, RN2.7, RN2.8, RN3.5, RN3.6, RN3.7, RN3.8, RN4.5, RN4.6, RN4.7, RN4.8, RN5.5, RN5.6, RN5.7, RN5.8, RN6.5, RN6.6, RN6.7, RN6.8; no longer R1.1, R10.1, R11.2, R12.1, R13.2, R14.1, R15.2, R16.2, R17.1, R18.2, R19.1, R2.2, R20.2, R3.1, R4.1, R5.2, R6.1, R7.2, R8.1, R9.2
Routing:
- net GND: track 0.00 -> 144.6 mm, vias 0 -> 1
- net VCC: track 0.00 -> 113.8 mm
- net N$20: track 0.00 -> 70.5 mm, vias 0 -> 1
- net N$18: track 0.00 -> 58.4 mm, vias 0 -> 1
- net N$2: track 0.00 -> 50.5 mm, vias 0 -> 1
- net N$4: track 0.00 -> 39.8 mm, vias 0 -> 1
- net N$16: track 0.00 -> 39.6 mm, vias 0 -> 1
- net N$6: track 0.00 -> 30.3 mm, vias 0 -> 1
- net N$14: track 0.00 -> 28.1 mm, vias 0 -> 1
- net N$9: track 0.00 -> 26.3 mm, vias 0 -> 1
- net N$8: track 0.00 -> 24.7 mm, vias 0 -> 1
- net N$22: track 0.00 -> 19.4 mm
- net N$1: track 0.00 -> 17.9 mm, vias 0 -> 1
- net N$7: track 0.00 -> 16.2 mm, vias 0 -> 1
- net N$12: track 0.00 -> 15.4 mm, vias 0 -> 1
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Other:
- board size 141 x 21.3 mm -> 102.5 x 17.5 mm

Commit message: hard level
Parts:
- removed JP1: (no value), pinhead:1X03
- added LED1: (no value), led:CHIPLED_0603
- moved JP2 5.93 mm to (-1.25, 7.84)
Connections:
- new net N$23: LED1.C, X1.1
- net GND: no longer JP1.3
- net N$21: now also LED1.A, RN3.4; no longer JP1.1, X1.1
- net VCC: no longer JP1.2
Routing:
- net GND: track 144.6 -> 91.7 mm, vias 1 -> 0
- net VCC: track 113.8 -> 74.5 mm
- net N$22: track 19.4 -> 0.00 mm
- net N$21: track 12.3 -> 0.00 mm
- net N$20: track 70.5 -> 72.7 mm
- net N$18: track 58.4 -> 60.4 mm
- net N$2: track 50.5 -> 52.2 mm
- net N$4: track 39.8 -> 41.3 mm
- net N$5: track 7.18 -> 6.09 mm
Other:
- board size 102.5 x 17.5 mm -> 99 x 17.8 mm

Commit message: done
Parts:
- moved LED1 11.8 mm to (5.77, -3.54), turned to 180 degrees
Routing:
- net GND: track 91.7 -> 138.8 mm, vias 0 -> 4
- net N$21: track 0.00 -> 30.5 mm
- net N$23: track 0.00 -> 16.9 mm, vias 0 -> 2
- net VCC: track 74.5 -> 87.1 mm
- net N$22: track 0.00 -> 10.1 mm, vias 0 -> 1
- net N$2: track 52.2 -> 56.2 mm
- net N$4: track 41.3 -> 43.0 mm
- net N$8: track 24.8 -> 26.0 mm
- net N$12: track 15.4 -> 14.5 mm
- net N$6: track 30.4 -> 29.8 mm
- net N$18: track 60.4 -> 59.8 mm
- net N$9: track 26.3 -> 26.9 mm
- added copper zone on layer 1, net GND
- added copper zone on layer 16, net GND
