File: pcb/lf.sch (EAGLE design)
At the start: 3 parts, among them IC1 TB6612FNG, IC2 TB6612FNG, U1 STM32F103RBT6

Commit message: sdsd
Other:
- moved on the sheet: IC1, IC2, U1
Changed lines of the file:
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@@
 <?xml version="1.0" encoding="utf-8"?>
 <!DOCTYPE eagle SYSTEM "eagle.dtd">
-<eagle version="7.1.0">
+<eagle version="8.1.1">
 <drawing>
 <settings>
@@
 <part name="IC1" library="tb6612" deviceset="TB6612FNG" device=""/>
 <part name="IC2" library="tb6612" deviceset="TB6612FNG" device=""/>
-<part name="U$1" library="PololuMG_v2" deviceset="POLOLU" device=""/>
 <part name="U1" library="STM32F103RBT6" deviceset="STM32F103RBT6" device=""/>
+<part name="GND1" library="supply1" deviceset="GND" device=""/>
+<part name="GND2" library="supply1" deviceset="GND" device=""/>
+<part name="GND3" library="supply1" deviceset="GND" device=""/>
+<part name="GND4" library="supply1" deviceset="GND" device=""/>
+<part name="GND5" library="supply1" deviceset="GND" device=""/>
+<part name="P+1" library="supply1" deviceset="VCC" device=""/>
+<part name="P+2" library="supply1" deviceset="VCC" device=""/>
+<part name="P+3" library="supply1" deviceset="VCC" device=""/>
+<part name="P+4" library="supply1" deviceset="VCC" device=""/>
+<part name="P+5" library="supply1" deviceset="VCC" device=""/>
+<part name="P+6" library="supply1" deviceset="VCC" device=""/>
 </parts>
 <sheets>
@@
 </plain>
 <instances>
-<instance part="IC1" gate="G$1" x="88.9" y="99.06"/>
-<instance part="IC2" gate="G$1" x="137.16" y="99.06"/>
-<instance part="U1" gate="A" x="109.22" y="228.6"/>
+<instance part="IC1" gate="G$1" x="200.66" y="269.24"/>
+<instance part="IC2" gate="G$1" x="200.66" y="208.28"/>
+<instance part="U1" gate="A" x="111.76" y="246.38"/>
+<instance part="GND1" gate="1" x="73.66" y="180.34"/>
+<instance part="GND2" gate="1" x="63.5" y="276.86"/>
+<instance part="GND3" gate="1" x="154.94" y="246.38"/>
+<instance part="GND4" gate="1" x="241.3" y="243.84"/>
+<instance part="GND5" gate="1" x="243.84" y="177.8"/>
+<instance part="P+1" gate="VCC" x="60.96" y="314.96"/>
+<instance part="P+2" gate="VCC" x="175.26" y="299.72"/>
+<instance part="P+3" gate="VCC" x="220.98" y="297.18"/>
+<instance part="P+4" gate="VCC" x="172.72" y="231.14"/>
+<instance part="P+5" gate="VCC" x="231.14" y="231.14"/>
+<instance part="P+6" gate="VCC" x="157.48" y="193.04"/>
 </instances>
 <busses>

Commit message: a takie tam poprawki
Parts:
- removed IC2: TB6612FNG, tb6612:TB6612FNG
- added JP1: (no value), pinhead:PINHD-1X6
- added JP2: (no value), pinhead:PINHD-1X3
- added JP3: (no value), pinhead:PINHD-1X4
- added JP4: (no value), pinhead:PINHD-1X2
- added U$1: 03-JST-B3B-XH-A, bt_con-jst-xh:03-JST-B3B-XH-A
- added U$4, U$5: 1X6, headers(2mm):1X6
- added X1: FH12-12S-0.5SH, con-hirose:FH12-12S-0.5SH
Connections:
- new net ADC0: U1.PA0-WKUP
- new net ADC1: U1.PA1
- new net ADC10: U1.PC0
- new net ADC11: U1.PC1
- new net ADC2: U1.PA2
- new net ADC3: U1.PA3
- new net ADC4: U1.PA4
- new net ADC5: U1.PA5
- new net ADC6: U1.PA6
- new net ADC7: U1.PA7
- new net BTLED: JP1.1
- new net ENC1A: U$4.3, U1.PB4
- new net ENC1B: U$4.2, U1.PB5
- new net ENC2A: U$5.3, U1.PB6
- new net ENC2B: U$5.2, U1.PB7
- new net GND: IC1.GND, IC1.PGND1@1, IC1.PGND1@2, IC1.PGND2@1, IC1.PGND2@2, JP1.5, JP2.2, JP3.4, JP4.2, U$4.1, U$5.1, U1.VSS_1, U1.VSS_2, U1.VSS_3, U1.VSS_4
- new net KEY: JP1.2
- new net LED0: U1.PB0
- new net LED1: U1.PB1
- new net LED2: U1.PB2
- new net LED3: U1.PB3
- new net LED4: U1.PC6
- new net LED5: U1.PC7
- new net LED6: U1.PC8
- new net LED7: U1.PC9
- new net M1A: IC1.AIN1, U1.PC2
- new net M1B: IC1.AIN2, U1.PC3
- new net M2A: IC1.BIN1, U1.PC4
- new net M2B: IC1.BIN2, U1.PC5
- new net MEN: IC1.!STBY, U1.PC10
- new net N$1: U1.PD0_OSC_IN
- new net N$2: U1.PD1_OSC_OUT
- new net N$3: U1.BOOT0
- new net N$6: IC1.AO2@1, IC1.AO2@2, U$4.5
- new net N$7: IC1.BO1@1, IC1.BO1@2, U$5.6
- new net N$8: IC1.BO2@1, IC1.BO2@2, U$5.5
- new net N$9: IC1.AO1@1, IC1.AO1@2, U$4.6
- new net PWM0: U1.PB13
- new net PWM1: IC1.PWMA, U1.PB14
- new net PWM2: IC1.PWMB, U1.PB15
- new net RXD: JP1.4, U1.PA9
- new net SCL: U1.PB11
- new net SDA: U1.PB10
- new net SW1: U1.PA11
- new net SW2: U1.PA12
- new net SWCLK: JP3.3, U1.PA14
- new net SWDIO: JP3.2, U1.PA13
- new net TXD: JP1.3, U1.PA10
- new net VCC: IC1.VCC, JP1.6, JP2.3, JP3.1, U$4.4, U$5.4, U1.VBAT, U1.VDD_1, U1.VDD_2, U1.VDD_3, U1.VDD_4
- new net VMOT: IC1.VM1, IC1.VM2, IC1.VM3, JP2.1, JP4.1

Commit message: schematic complete
Parts:
- added C1, C3, C4: (no value), rcl:C-EUC0603K
- added C5, C6: 100n, rcl:C-EUC0603K
- added C8: (no value), rcl:CPOL-EUC/6032-28R
- added L1: (no value), rcl:L-EUL3216C
- added LED1, LED10, LED11, LED12, LED2, LED3, LED4, LED5, LED6, LED7, LED8, LED9: (no value), led:LEDCHIPLED_0603
- added MOSFET: FDN360P, transistor-power:FDN360P
- added Q1: (no value), crystal-geyer_V1_0:KX-7
- added R1, R16, R17, R18, R19: (no value), rcl:R-EU_R0603
- added R14: 4k7, rcl:R-EU_R0603
- added R15: 100R, rcl:R-EU_R0603
- added R2, R3, R5: 10k, rcl:R-EU_R0603
- added R4: 100, rcl:R-EU_R0603
- added RN1, RN2, RN3: (no value), resistor-dil:4R-NEXB28V
- added S1: (no value), switch:255SB
- added S3: (no value), SparkFun-Switches:MOMENTARY-SWITCH-SPST-2-SMD-5.2MM
- X1: value FH12-12S-0.5SH -> FH12-14S-0.5SH; device con-hirose:FH12-12S-0.5SH -> con-hirose:FH12-14S-0.5SH
Connections:
- removed net SW2: U1.PA12
- new net ADC12: R18.2, R19.1
- new net ADC13: R16.1, R17.2
- new net ADC8: X1-11.1
- new net ADC9: X1-12.1
- new net LED8: LED9.A, U1.PC10
- new net LED9: LED10.A, U1.PC11
- new net N$10: C3.1, Q1.2, R1.2, U1.PD0_OSC_IN
- new net N$11: C5.2, R3.2, U1.NRST
- new net N$12: JP4.1, S1.S
- new net N$13: R18.1, U$1-1.1
- new net N$14: R17.1, U$1-2.1
- new net N$15: LED1.C, RN1A.2
- new net N$16: LED2.C, RN1B.2
- new net N$17: LED3.C, RN1C.2
- new net N$18: LED4.C, RN1D.2
- new net N$19: LED5.C, RN2A.2
- new net N$20: LED6.C, RN2B.2
- new net N$21: LED7.C, RN2C.2
- new net N$22: LED8.C, RN2D.2
- new net N$23: LED9.C, RN3A.2
- new net N$24: LED10.C, RN3B.2
- new net N$25: LED11.C, RN3C.2
- new net N$26: LED12.C, RN3D.2
- new net N$27: MOSFET.G, R4.1, R5.1
- new net N$28: MOSFET.S, X1-1.1
- new net N$4: C6.2, U1.VSSA
- new net N$5: C1.2, R15.1
- new net SENSOREN: R4.2, U1.PA8
- new net STLED: LED11.A, U1.PB12
- net ADC0: now also X1-3.1
- net ADC1: now also X1-4.1
- net ADC10: now also X1-13.1
- net ADC11: now also X1-14.1
- net ADC2: now also X1-5.1
- net ADC3: now also X1-6.1
- net ADC4: now also X1-7.1
- net ADC5: now also X1-8.1
- net ADC6: now also X1-9.1
- net ADC7: now also X1-10.1
- net GND: now also C3.2, C4.2, C5.1, C8.-, R15.2, R16.2, R19.2, R2.2, RN1A.1, RN1B.1, RN1C.1, RN1D.1, RN2A.1, RN2B.1, RN2C.1, RN2D.1, RN3A.1, RN3B.1, RN3C.1, RN3D.1, S3.1, S3.2, U$1-3.1, X1-2.1
- net LED0: now also LED1.A
- net LED1: now also LED2.A
- net LED2: now also LED3.A
- net LED3: now also LED4.A
- net LED4: now also LED5.A
- net LED5: now also LED6.A
- net LED6: now also LED7.A
- net LED7: now also LED8.A
- net MEN: now also U1.PC12; no longer U1.PC10
- net N$1: now also C4.1, Q1.1, R1.1, U1.PD1_OSC_OUT; no longer U1.PD0_OSC_IN
- net N$2: now also C6.1, L1.2, U1.VDDA; no longer U1.PD1_OSC_OUT
- net N$3: now also R2.1
- net SW1: now also C1.1, R14.1, S3.3, S3.4, U1.PC13-TAMPER-RTC; no longer U1.PA11
- net VCC: now also L1.1, LED12.A, MOSFET.D, R14.2, R3.1, R5.2
- net VMOT: now also C8.+, S1.P; no longer JP4.1
Other:
- moved on the sheet: U$1-1, U$1-2, U$1-3, X1-1, X1-10, X1-11, X1-12, X1-2, X1-3, X1-4, X1-5, X1-6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

Commit message: o już niewiele
Parts:
- removed JP4: (no value), pinhead:PINHD-1X2
- removed S1: (no value), switch:255SB
- added S2: (no value), SparkFun-Switches:SWITCH-SPDT-PTH-11.6X4.0MM
Connections:
- removed net N$13: R18.1, U$1-1.1
- net GND: no longer JP4.2
- net N$12: now also R18.1, S2.S, U$1-1.1; no longer JP4.1, S1.S
- net VMOT: now also S2.P; no longer S1.P
Changed lines of the file:
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@@
 <part name="JP2" library="pinhead" deviceset="PINHD-1X3" device=""/>
 <part name="JP3" library="pinhead" deviceset="PINHD-1X4" device=""/>
-<part name="JP4" library="pinhead" deviceset="PINHD-1X2" device=""/>
 <part name="JP1" library="pinhead" deviceset="PINHD-1X6" device=""/>
 <part name="GND6" library="supply1" deviceset="GND" device=""/>
@@
 <part name="GND5" library="supply1" deviceset="GND" device=""/>
 <part name="L1" library="rcl" deviceset="L-EU" device="L3216C"/>
-<part name="S1" library="switch" deviceset="255SB" device=""/>
 <part name="S3" library="SparkFun-Switches" deviceset="MOMENTARY-SWITCH-SPST-2" device="-SMD-5.2MM"/>
 <part name="P+6" library="supply1" deviceset="VCC" device=""/>
@@
 <part name="X1" library="con-hirose" deviceset="FH12-14S-0.5S" device="H"/>
 <part name="GND16" library="supply1" deviceset="GND" device=""/>
+<part name="S2" library="SparkFun-Switches" deviceset="SWITCH-SPDT" device="-PTH-11.6X4.0MM"/>
 </parts>
 <sheets>
@@
 <instance part="JP2" gate="A" x="27.94" y="312.42" rot="MR0"/>
 <instance part="JP3" gate="A" x="30.48" y="241.3" rot="MR0"/>
-<instance part="JP4" gate="G$1" x="27.94" y="325.12" rot="MR0"/>
 <instance part="JP1" gate="A" x="30.48" y="266.7" rot="R180"/>
 <instance part="GND6" gate="1" x="45.72" y="233.68"/>
@@
 <instance part="GND5" gate="1" x="45.72" y="281.94"/>
 <instance part="L1" gate="G$1" x="68.58" y="302.26" rot="R90"/>
-<instance part="S1" gate="1" x="60.96" y="335.28"/>
 <instance part="S3" gate="G$1" x="309.88" y="281.94" rot="R90"/>
 <instance part="P+6" gate="VCC" x="157.48" y="256.54"/>
@@
 <instance part="X1" gate="-14" x="205.74" y="320.04"/>
 <instance part="GND16" gate="1" x="177.8" y="345.44"/>
+<instance part="S2" gate="1" x="63.5" y="335.28" rot="R90"/>
 </instances>
 <busses>
@@
 </segment>
 <segment>
-<pinref part="JP4" gate="G$1" pin="2"/>
-<wire x1="30.48" y1="325.12" x2="43.18" y2="325.12" width="0.1524" layer="91"/>
-<wire x1="43.18" y1="325.12" x2="43.18" y2="312.42" width="0.1524" layer="91"/>
 <pinref part="JP2" gate="A" pin="2"/>
 <wire x1="43.18" y1="312.42" x2="30.48" y2="312.42" width="0.1524" layer="91"/>
 <pinref part="GND7" gate="1" pin="GND"/>
 <wire x1="43.18" y1="312.42" x2="43.18" y2="304.8" width="0.1524" layer="91"/>
-<junction x="43.18" y="312.42"/>
 </segment>
 <segment>
@@
 <wire x1="38.1" y1="314.96" x2="30.48" y2="314.96" width="0.1524" layer="91"/>
 <label x="38.1" y="327.66" size="1.27" layer="95" xref="yes"/>
-<pinref part="S1" gate="1" pin="P"/>
 <wire x1="63.5" y1="330.2" x2="38.1" y2="330.2" width="0.1524" layer="91"/>
+<pinref part="S2" gate="1" pin="P"/>
+<wire x1="63.5" y1="330.2" x2="63.5" y2="332.74" width="0.1524" layer="91"/>
 </segment>
 <segment>
@@
 <net name="N$12" class="0">
 <segment>
-<pinref part="JP4" gate="G$1" pin="1"/>
-<wire x1="30.48" y1="327.66" x2="35.56" y2="327.66" width="0.1524" layer="91"/>
-<wire x1="35.56" y1="327.66" x2="35.56" y2="337.82" width="0.1524" layer="91"/>
-<wire x1="35.56" y1="337.82" x2="53.34" y2="337.82" width="0.1524" layer="91"/>
-<wire x1="53.34" y1="337.82" x2="53.34" y2="342.9" width="0.1524" layer="91"/>
-<wire x1="53.34" y1="342.9" x2="66.04" y2="342.9" width="0.1524" layer="91"/>
-<pinref part="S1" gate="1" pin="S"/>
 <wire x1="66.04" y1="342.9" x2="66.04" y2="340.36" width="0.1524" layer="91"/>
+<pinref part="U$1" gate="-1" pin="1"/>
+<pinref part="R18" gate="G$1" pin="1"/>
+<wire x1="121.92" y1="332.74" x2="116.84" y2="332.74" width="0.1524" layer="91"/>
+<wire x1="116.84" y1="332.74" x2="114.3" y2="332.74" width="0.1524" layer="91"/>
+<wire x1="66.04" y1="342.9" x2="116.84" y2="342.9" width="0.1524" layer="91"/>
+<wire x1="116.84" y1="342.9" x2="116.84" y2="332.74" width="0.1524" layer="91"/>
+<junction x="116.84" y="332.74"/>
+<pinref part="S2" gate="1" pin="S"/>
 </segment>
 </net>
@@
 </segment>
 </net>
-<net name="N$13" class="0">
-<segment>
-<pinref part="U$1" gate="-1" pin="1"/>
-<pinref part="R18" gate="G$1" pin="1"/>
-<wire x1="121.92" y1="332.74" x2="114.3" y2="332.74" width="0.1524" layer="91"/>
-</segment>
-</net>

Commit message: hard level
Connections:
- removed net PWM0: U1.PB13
- removed net SCL: U1.PB11
- removed net SDA: U1.PB10
- net ADC10: now also U1.PC1; no longer U1.PC0
- net ADC11: now also U1.PC0; no longer U1.PC1
- net ADC8: now also U1.PB0
- net ADC9: now also U1.PB1
- net ENC2A: now also U1.PB7; no longer U1.PB6
- net ENC2B: now also U1.PB6; no longer U1.PB7
- net LED0: now also U1.PB10; no longer U1.PB0
- net LED1: now also U1.PB11; no longer U1.PB1
- net LED2: now also U1.PB12; no longer U1.PB2
- net LED3: now also U1.PB13; no longer U1.PB3
- net LED8: now also U1.PA8; no longer U1.PC10
- net LED9: now also U1.PA11; no longer U1.PC11
- net SENSOREN: now also U1.PB2; no longer U1.PA8
- net STLED: now also U1.PA12; no longer U1.PB12

Commit message: już końcówka
Parts:
- removed L1: (no value), rcl:L-EUL3216C
Connections:
- removed net N$2: C6.1, L1.2, U1.VDDA
- net VCC: now also C6.1, U1.VDDA; no longer L1.1
Changed lines of the file:
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@@
 <part name="C8" library="rcl" deviceset="CPOL-EU" device="C/6032-28R"/>
 <part name="GND5" library="supply1" deviceset="GND" device=""/>
-<part name="L1" library="rcl" deviceset="L-EU" device="L3216C"/>
 <part name="S3" library="SparkFun-Switches" deviceset="MOMENTARY-SWITCH-SPST-2" device="-SMD-5.2MM"/>
 <part name="P+6" library="supply1" deviceset="VCC" device=""/>
@@
 <instance part="C8" gate="G$1" x="236.22" y="294.64"/>
 <instance part="GND5" gate="1" x="45.72" y="281.94"/>
-<instance part="L1" gate="G$1" x="68.58" y="302.26" rot="R90"/>
 <instance part="S3" gate="G$1" x="309.88" y="281.94" rot="R90"/>
 <instance part="P+6" gate="VCC" x="157.48" y="256.54"/>
@@
 <wire x1="63.5" y1="287.02" x2="63.5" y2="292.1" width="0.1524" layer="91"/>
 <junction x="63.5" y="292.1"/>
-<pinref part="L1" gate="G$1" pin="1"/>
+<pinref part="U1" gate="A" pin="VDDA"/>
+<pinref part="C6" gate="G$1" pin="1"/>
+<wire x1="76.2" y1="302.26" x2="81.28" y2="302.26" width="0.1524" layer="91"/>
+<wire x1="66.04" y1="185.42" x2="71.12" y2="185.42" width="0.1524" layer="91"/>
+<wire x1="71.12" y1="185.42" x2="71.12" y2="195.58" width="0.1524" layer="91"/>
+<wire x1="71.12" y1="195.58" x2="76.2" y2="195.58" width="0.1524" layer="91"/>
+<wire x1="76.2" y1="195.58" x2="76.2" y2="302.26" width="0.1524" layer="91"/>
+<junction x="76.2" y="302.26"/>
+<wire x1="76.2" y1="302.26" x2="63.5" y2="302.26" width="0.1524" layer="91"/>
 <junction x="63.5" y="302.26"/>
 </segment>
@@
 </segment>
 </net>
-<net name="N$2" class="0">
-<segment>
-<pinref part="U1" gate="A" pin="VDDA"/>
-<pinref part="L1" gate="G$1" pin="2"/>
-<wire x1="73.66" y1="302.26" x2="76.2" y2="302.26" width="0.1524" layer="91"/>
-<pinref part="C6" gate="G$1" pin="1"/>
-<wire x1="76.2" y1="302.26" x2="81.28" y2="302.26" width="0.1524" layer="91"/>
-<wire x1="66.04" y1="185.42" x2="71.12" y2="185.42" width="0.1524" layer="91"/>
-<wire x1="71.12" y1="185.42" x2="71.12" y2="195.58" width="0.1524" layer="91"/>
-<wire x1="71.12" y1="195.58" x2="76.2" y2="195.58" width="0.1524" layer="91"/>
-<wire x1="76.2" y1="195.58" x2="76.2" y2="302.26" width="0.1524" layer="91"/>
-<junction x="76.2" y="302.26"/>
-</segment>
-</net>

Commit message: done
Other:
- moved on the sheet: C1, R14, R15, S3
Changed lines of the file:
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@@
 <part name="GND16" library="supply1" deviceset="GND" device=""/>
 <part name="S2" library="SparkFun-Switches" deviceset="SWITCH-SPDT" device="-PTH-11.6X4.0MM"/>
+<part name="FRAME1" library="frames" deviceset="A3L-LOC" device=""/>
 </parts>
 <sheets>
@@
 <instance part="R2" gate="G$1" x="55.88" y="284.48" rot="R180"/>
 <instance part="R3" gate="G$1" x="157.48" y="246.38" rot="R270"/>
-<instance part="R14" gate="G$1" x="317.5" y="294.64" rot="R90"/>
-<instance part="R15" gate="G$1" x="320.04" y="274.32" rot="R180"/>
-<instance part="GND10" gate="1" x="312.42" y="266.7"/>
-<instance part="P+9" gate="VCC" x="317.5" y="307.34"/>
+<instance part="R14" gate="G$1" x="248.92" y="337.82" rot="R90"/>
+<instance part="R15" gate="G$1" x="251.46" y="317.5" rot="R180"/>
+<instance part="GND10" gate="1" x="243.84" y="309.88"/>
+<instance part="P+9" gate="VCC" x="248.92" y="350.52"/>
 <instance part="GND14" gate="1" x="210.82" y="187.96"/>
-<instance part="C1" gate="G$1" x="325.12" y="281.94"/>
+<instance part="C1" gate="G$1" x="256.54" y="325.12"/>
 <instance part="C3" gate="G$1" x="162.56" y="269.24" rot="R90"/>
 <instance part="C4" gate="G$1" x="162.56" y="259.08" rot="R90"/>
@@
 <instance part="C8" gate="G$1" x="236.22" y="294.64"/>
 <instance part="GND5" gate="1" x="45.72" y="281.94"/>
-<instance part="S3" gate="G$1" x="309.88" y="281.94" rot="R90"/>
+<instance part="S3" gate="G$1" x="241.3" y="325.12" rot="R90"/>
 <instance part="P+6" gate="VCC" x="157.48" y="256.54"/>
 <instance part="GND11" gate="1" x="157.48" y="226.06"/>
@@
 <instance part="GND16" gate="1" x="177.8" y="345.44"/>
 <instance part="S2" gate="1" x="63.5" y="335.28" rot="R90"/>
+<instance part="FRAME1" gate="G$1" x="-38.1" y="134.62"/>
 </instances>
 <busses>
@@
 <pinref part="GND10" gate="1" pin="GND"/>
 <pinref part="S3" gate="G$1" pin="2"/>
-<wire x1="312.42" y1="269.24" x2="312.42" y2="274.32" width="0.1524" layer="91"/>
+<wire x1="243.84" y1="312.42" x2="243.84" y2="317.5" width="0.1524" layer="91"/>
 <pinref part="R15" gate="G$1" pin="2"/>
-<wire x1="312.42" y1="274.32" x2="312.42" y2="276.86" width="0.1524" layer="91"/>
-<wire x1="314.96" y1="274.32" x2="312.42" y2="274.32" width="0.1524" layer="91"/>
-<junction x="312.42" y="274.32"/>
+<wire x1="243.84" y1="317.5" x2="243.84" y2="320.04" width="0.1524" layer="91"/>
+<wire x1="246.38" y1="317.5" x2="243.84" y2="317.5" width="0.1524" layer="91"/>
+<junction x="243.84" y="317.5"/>
 <pinref part="S3" gate="G$1" pin="1"/>
-<wire x1="309.88" y1="276.86" x2="309.88" y2="274.32" width="0.1524" layer="91"/>
-<wire x1="309.88" y1="274.32" x2="312.42" y2="274.32" width="0.1524" layer="91"/>
+<wire x1="241.3" y1="320.04" x2="241.3" y2="317.5" width="0.1524" layer="91"/>
+<wire x1="241.3" y1="317.5" x2="243.84" y2="317.5" width="0.1524" layer="91"/>
 </segment>
 <segment>
@@
 <pinref part="R14" gate="G$1" pin="2"/>
 <pinref part="P+9" gate="VCC" pin="VCC"/>
-<wire x1="317.5" y1="299.72" x2="317.5" y2="304.8" width="0.1524" layer="91"/>
+<wire x1="248.92" y1="342.9" x2="248.92" y2="347.98" width="0.1524" layer="91"/>
 </segment>
 <segment>
@@
 <pinref part="R15" gate="G$1" pin="1"/>
 <pinref part="C1" gate="G$1" pin="2"/>
-<wire x1="325.12" y1="274.32" x2="325.12" y2="276.86" width="0.1524" layer="91"/>
+<wire x1="256.54" y1="317.5" x2="256.54" y2="320.04" width="0.1524" layer="91"/>
 </segment>
 </net>
@@
 <segment>
 <pinref part="C1" gate="G$1" pin="1"/>
-<wire x1="325.12" y1="284.48" x2="325.12" y2="289.56" width="0.1524" layer="91"/>
+<wire x1="256.54" y1="327.66" x2="256.54" y2="332.74" width="0.1524" layer="91"/>
 <pinref part="R14" gate="G$1" pin="1"/>
-<wire x1="325.12" y1="289.56" x2="317.5" y2="289.56" width="0.1524" layer="91"/>
-<wire x1="317.5" y1="289.56" x2="312.42" y2="289.56" width="0.1524" layer="91"/>
-<junction x="317.5" y="289.56"/>
+<wire x1="256.54" y1="332.74" x2="248.92" y2="332.74" width="0.1524" layer="91"/>
+<wire x1="248.92" y1="332.74" x2="243.84" y2="332.74" width="0.1524" layer="91"/>
+<junction x="248.92" y="332.74"/>
 <pinref part="S3" gate="G$1" pin="4"/>
-<wire x1="312.42" y1="289.56" x2="312.42" y2="287.02" width="0.1524" layer="91"/>
-<wire x1="312.42" y1="289.56" x2="309.88" y2="289.56" width="0.1524" layer="91"/>
-<junction x="312.42" y="289.56"/>
+<wire x1="243.84" y1="332.74" x2="243.84" y2="330.2" width="0.1524" layer="91"/>
+<wire x1="243.84" y1="332.74" x2="241.3" y2="332.74" width="0.1524" layer="91"/>
+<junction x="243.84" y="332.74"/>
 <pinref part="S3" gate="G$1" pin="3"/>
-<wire x1="309.88" y1="289.56" x2="309.88" y2="287.02" width="0.1524" layer="91"/>
-<wire x1="309.88" y1="289.56" x2="299.72" y2="289.56" width="0.1524" layer="91"/>
-<junction x="309.88" y="289.56"/>
-<label x="299.72" y="289.56" size="1.27" layer="95" rot="R180" xref="yes"/>
-</segment>
-</net>
+<wire x1="241.3" y1="332.74" x2="241.3" y2="330.2" width="0.1524" layer="91"/>
+<wire x1="241.3" y1="332.74" x2="231.14" y2="332.74" width="0.1524" layer="91"/>
+<junction x="241.3" y="332.74"/>
+<label x="231.14" y="332.74" size="1.27" layer="95" rot="R180" xref="yes"/>
+</segment>
+</net>

Commit message: part_values
Parts:
- Q1: value (none) -> 8MHz
- R1: value (none) -> 1M
Changed lines of the file:
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@@
 <?xml version="1.0" encoding="utf-8"?>
 <!DOCTYPE eagle SYSTEM "eagle.dtd">
-<eagle version="8.1.1">
+<eagle version="7.7.0">
 <drawing>
 <settings>
@@
 <part name="P+5" library="supply1" deviceset="VCC" device=""/>
 <part name="P+8" library="supply1" deviceset="VCC" device=""/>
-<part name="Q1" library="crystal-geyer_V1_0" deviceset="KX" device="-7"/>
-<part name="R1" library="rcl" deviceset="R-EU_" device="R0603"/>
+<part name="Q1" library="crystal-geyer_V1_0" deviceset="KX" device="-7" value="8MHz"/>
+<part name="R1" library="rcl" deviceset="R-EU_" device="R0603" value="1M"/>
 <part name="R2" library="rcl" deviceset="R-EU_" device="R0603" value="10k"/>
 <part name="R3" library="rcl" deviceset="R-EU_" device="R0603" value="10k"/>
