File: pcb/lf.sch (EAGLE design)
At the start: 45 parts, among them IC1 TB6612FNG, Q1 8MHz, U1 STM32F103RBT6, X1 FH12-14S-0.5SH

Commit message: cubemx
Parts:
- Q1: value 8MHz -> 16MHz
Changed lines of the file:
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@@
 <part name="P+5" library="supply1" deviceset="VCC" device=""/>
 <part name="P+8" library="supply1" deviceset="VCC" device=""/>
-<part name="Q1" library="crystal-geyer_V1_0" deviceset="KX" device="-7" value="8MHz"/>
+<part name="Q1" library="crystal-geyer_V1_0" deviceset="KX" device="-7" value="16MHz"/>
 <part name="R1" library="rcl" deviceset="R-EU_" device="R0603" value="1M"/>
 <part name="R2" library="rcl" deviceset="R-EU_" device="R0603" value="10k"/>
