File: pcb/lf.brd (EAGLE design)
At the start: 160 x 27.6 mm, 5 parts, among them IC1 TB6612FNG, IC2 TB6612FNG, U1 STM32F103RBT6

Commit message: a takie tam poprawki
Parts:
- removed IC2: TB6612FNG, tb6612:SSOP24
- added JP1: (no value), pinhead:1X06
- added JP2: (no value), pinhead:1X03
- added JP3: (no value), pinhead:1X04
- added JP4: (no value), pinhead:1X02
- added U$1: 03-JST-B3B-XH-A, bt_con-jst-xh:B3B-XH
- added U$4, U$5: 1X6, headers(2mm):1X6
- added X1: FH12-12S-0.5SH, con-hirose:FH12-12S-0.5SH
- turned U1 to 45 degrees
Connections:
- removed net VDD_1: U1.32
- removed net VDD_2: U1.48
- removed net VDD_3: U1.64
- removed net VDD_4: U1.19
- new net ADC0: U1.14
- new net ADC1: U1.15
- new net ADC10: U1.8
- new net ADC11: U1.9
- new net ADC2: U1.16
- new net ADC3: U1.17
- new net ADC4: U1.20
- new net ADC5: U1.21
- new net ADC6: U1.22
- new net ADC7: U1.23
- new net BTLED: JP1.1
- new net ENC1A: U$4.3, U1.56
- new net ENC1B: U$4.2, U1.57
- new net ENC2A: U$5.3, U1.58
- new net ENC2B: U$5.2, U1.59
- new net GND: IC1.10, IC1.18, IC1.3, IC1.4, IC1.9, JP1.5, JP2.2, JP3.4, JP4.2, U$4.1, U$5.1, U1.18, U1.31, U1.47, U1.63
- new net KEY: JP1.2
- new net LED0: U1.26
- new net LED1: U1.27
- new net LED2: U1.28
- new net LED3: U1.55
- new net LED4: U1.37
- new net LED5: U1.38
- new net LED6: U1.39
- new net LED7: U1.40
- new net M1A: IC1.21, U1.10
- new net M1B: IC1.22, U1.11
- new net M2A: IC1.17, U1.24
- new net M2B: IC1.16, U1.25
- new net MEN: IC1.19, U1.51
- new net N$1: U1.5
- new net N$2: U1.6
- new net N$3: U1.60
- new net N$6: IC1.5, IC1.6, U$4.5
- new net N$7: IC1.11, IC1.12, U$5.6
- new net N$8: IC1.7, IC1.8, U$5.5
- new net N$9: IC1.1, IC1.2, U$4.6
- new net PWM0: U1.34
- new net PWM1: IC1.23, U1.35
- new net PWM2: IC1.15, U1.36
- new net RXD: JP1.4, U1.42
- new net SCL: U1.30
- new net SDA: U1.29
- new net SW1: U1.44
- new net SW2: U1.45
- new net SWCLK: JP3.3, U1.49
- new net SWDIO: JP3.2, U1.46
- new net TXD: JP1.3, U1.43
- new net VCC: IC1.20, JP1.6, JP2.3, JP3.1, U$4.4, U$5.4, U1.1, U1.19, U1.32, U1.48, U1.64
- new net VMOT: IC1.13, IC1.14, IC1.24, JP2.1, JP4.1

Commit message: schematic complete
Parts:
- added C1, C3, C4: (no value), rcl:C0603K
- added C5, C6: 100n, rcl:C0603K
- added C8: (no value), rcl:C/6032-28R
- added L1: (no value), rcl:L3216C
- added LED1, LED10, LED11, LED12, LED2, LED3, LED4, LED5, LED6, LED7, LED8, LED9: (no value), led:CHIPLED_0603
- added MOSFET: FDN360P, transistor-power:SUPER-SOT3
- added Q1: (no value), crystal-geyer_V1_0:3.2X2.5_KX-7
- added R1, R16, R17, R18, R19: (no value), rcl:R0603
- added R14: 4k7, rcl:R0603
- added R15: 100R, rcl:R0603
- added R2, R3, R5: 10k, rcl:R0603
- added R4: 100, rcl:R0603
- added RN1, RN2, RN3: (no value), resistor-dil:EXB28V
- added S1: (no value), switch:255SB
- added S3: (no value), SparkFun-Switches:TACTILE_SWITCH_SMD_5.2MM
- X1: value FH12-12S-0.5SH -> FH12-14S-0.5SH; device con-hirose:FH12-12S-0.5SH -> con-hirose:FH12-14S-0.5SH
- moved X1 1.80 mm to (52.1, 25.4)
Connections:
- removed net SW2: U1.45
- removed net VDDA: U1.13
- new net ADC12: R18.2, R19.1
- new net ADC13: R16.1, R17.2
- new net ADC8: X1.11
- new net ADC9: X1.12
- new net LED8: LED9.A, U1.51
- new net LED9: LED10.A, U1.52
- new net N$10: C3.1, Q1.3, R1.2, U1.5
- new net N$11: C5.2, R3.2, U1.7
- new net N$12: JP4.1, S1.3
- new net N$13: R18.1, U$1.P$1
- new net N$14: R17.1, U$1.P$2
- new net N$15: LED1.C, RN1.8
- new net N$16: LED2.C, RN1.7
- new net N$17: LED3.C, RN1.6
- new net N$18: LED4.C, RN1.5
- new net N$19: LED5.C, RN2.8
- new net N$20: LED6.C, RN2.7
- new net N$21: LED7.C, RN2.6
- new net N$22: LED8.C, RN2.5
- new net N$23: LED9.C, RN3.8
- new net N$24: LED10.C, RN3.7
- new net N$25: LED11.C, RN3.6
- new net N$26: LED12.C, RN3.5
- new net N$27: MOSFET.1, R4.1, R5.1
- new net N$28: MOSFET.2, X1.1
- new net N$4: C6.2, U1.12
- new net N$5: C1.2, R15.1
- new net SENSOREN: R4.2, U1.41
- new net STLED: LED11.A, U1.33
- net ADC0: now also X1.3
- net ADC1: now also X1.4
- net ADC10: now also X1.13
- net ADC11: now also X1.14
- net ADC2: now also X1.5
- net ADC3: now also X1.6
- net ADC4: now also X1.7
- net ADC5: now also X1.8
- net ADC6: now also X1.9
- net ADC7: now also X1.10
- net GND: now also C3.2, C4.2, C5.1, C8.-, R15.2, R16.2, R19.2, R2.2, RN1.1, RN1.2, RN1.3, RN1.4, RN2.1, RN2.2, RN2.3, RN2.4, RN3.1, RN3.2, RN3.3, RN3.4, S3.1, S3.2, U$1.P$3, X1.2
- net LED0: now also LED1.A
- net LED1: now also LED2.A
- net LED2: now also LED3.A
- net LED3: now also LED4.A
- net LED4: now also LED5.A
- net LED5: now also LED6.A
- net LED6: now also LED7.A
- net LED7: now also LED8.A
- net MEN: now also U1.53; no longer U1.51
- net N$1: now also C4.1, Q1.1, R1.1, U1.6; no longer U1.5
- net N$2: now also C6.1, L1.2, U1.13; no longer U1.6
- net N$3: now also R2.1
- net SW1: now also C1.1, R14.1, S3.3, S3.4, U1.2; no longer U1.44
- net VCC: now also L1.1, LED12.A, MOSFET.3, R14.2, R3.1, R5.2
- net VMOT: now also C8.+, S1.2; no longer JP4.1

Commit message: o już niewiele
Parts:
- removed JP4: (no value), pinhead:1X02
- removed S1: (no value), switch:255SB
- removed U$2, U$3: (no value), PololuMG_v2:HP_NM
- added S2: (no value), SparkFun-Switches:SWITCH_SPDT_PTH_11.6X4.0MM
- moved S3 67.7 mm to (55.5, 3.19), turned to 90 degrees
- moved LED12 62.0 mm to (55.2, 17.9), turned to 180 degrees
- moved LED11 60.9 mm to (53.7, 17.9), turned to 180 degrees
- moved RN3 59.3 mm to (51.5, 14.3)
- moved LED10 58.8 mm to (50.8, 17.9), turned to 180 degrees
- moved LED9 57.7 mm to (49.3, 17.9), turned to 180 degrees
- moved LED8 56.6 mm to (47.9, 17.9), turned to 180 degrees
- moved LED7 55.6 mm to (46.4, 17.9), turned to 180 degrees
- moved RN2 55.3 mm to (45.3, 14.3)
- moved LED6 54.5 mm to (44.9, 17.9), turned to 180 degrees
- moved LED5 53.4 mm to (43.5, 17.9), turned to 180 degrees
- moved LED4 52.3 mm to (42.0, 17.9), turned to 180 degrees
- moved LED3 51.3 mm to (40.6, 17.9), turned to 180 degrees
- moved LED2 50.2 mm to (39.1, 17.9), turned to 180 degrees
- moved RN1 49.4 mm to (39.9, 14.3)
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Connections:
- removed net N$13: R18.1, U$1.P$1
- net GND: no longer JP4.2
- net N$12: now also R18.1, S2.3, U$1.P$1; no longer JP4.1, S1.3
- net VMOT: now also S2.2; no longer S1.2
Other:
- board size 160 x 27.6 mm -> 140 x 37 mm

Commit message: hard level
Parts:
- moved C8 18.5 mm to (79.6, 6.00), turned to 0 degrees
- moved R17 12.0 mm to (92.7, 5.84)
- moved R15 11.3 mm to (50.5, 3.99), turned to 0 degrees
- moved R16 10.5 mm to (90.2, 5.83)
- moved R19 10.4 mm to (87.8, 5.84)
- moved C1 9.57 mm to (50.7, 5.84), turned to 180 degrees
- moved C5 9.42 mm to (77.4, 28.5), turned to 270 degrees
- moved C3 9.16 mm to (84.1, 28.6), turned to 270 degrees
- moved R18 7.31 mm to (85.7, 5.83)
- moved IC1 5.52 mm to (93.5, 15.6)
- moved RN2 5.25 mm to (45.6, 9.08)
- moved RN1 5.24 mm to (39.7, 9.08)
- moved RN3 5.24 mm to (51.6, 9.08)
- moved R3 4.73 mm to (83.2, 22.7), turned to 180 degrees
- moved R1 4.67 mm to (82.1, 25.4), turned to 0 degrees
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Connections:
- removed net PWM0: U1.34
- removed net SCL: U1.30
- removed net SDA: U1.29
- net ADC10: now also U1.9; no longer U1.8
- net ADC11: now also U1.8; no longer U1.9
- net ADC8: now also U1.26
- net ADC9: now also U1.27
- net ENC2A: now also U1.59; no longer U1.58
- net ENC2B: now also U1.58; no longer U1.59
- net LED0: now also U1.29; no longer U1.26
- net LED1: now also U1.30; no longer U1.27
- net LED2: now also U1.33; no longer U1.28
- net LED3: now also U1.34; no longer U1.55
- net LED8: now also U1.41; no longer U1.51
- net LED9: now also U1.44; no longer U1.52
- net SENSOREN: now also U1.28; no longer U1.41
- net STLED: now also U1.45; no longer U1.33
Routing:
- net GND: track 0.00 -> 130.0 mm, vias 0 -> 3
- net VCC: track 0.00 -> 81.9 mm
- net N$6: track 0.00 -> 76.5 mm, vias 0 -> 1
- net N$9: track 0.00 -> 68.1 mm, vias 0 -> 1
- net ENC1B: track 0.00 -> 54.2 mm, vias 0 -> 1
- net ENC1A: track 0.00 -> 52.1 mm, vias 0 -> 1
- net M2B: track 0.00 -> 49.2 mm, vias 0 -> 2
- net M2A: track 0.00 -> 46.4 mm, vias 0 -> 2
- net ENC2A: track 0.00 -> 44.1 mm, vias 0 -> 2
- net ENC2B: track 0.00 -> 43.4 mm, vias 0 -> 2
- net VMOT: track 0.00 -> 40.2 mm
- net PWM2: track 0.00 -> 40.1 mm, vias 0 -> 2
- net PWM1: track 0.00 -> 38.3 mm, vias 0 -> 2
- net MEN: track 0.00 -> 36.2 mm, vias 0 -> 4
- net N$8: track 0.00 -> 28.8 mm, vias 0 -> 1
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
Commit message: już końcówka
Parts:
- removed L1: (no value), rcl:L3216C
- moved C3 6.09 mm to (78.1, 29.4), turned to 180 degrees
- moved LED12 5.91 mm to (55.8, 9.45), turned to 90 degrees
- moved R3 5.02 mm to (78.3, 23.7), turned to 90 degrees
- moved LED11 2.25 mm to (51.5, 15.6)
- moved C4 1.31 mm to (78.6, 27.2)
- moved C5 1.28 mm to (77.3, 27.2)
- moved Q1 1.28 mm to (81.3, 27.1)
- moved R1 1.24 mm to (81.3, 24.5)
- moved R15 1.16 mm to (50.8, 5.10)
- moved C1 0.97 mm to (50.9, 6.79)
- moved R2 0.95 mm to (80.3, 17.3)
- moved LED3 0.71 mm to (39.9, 15.6)
- moved LED4 0.71 mm to (41.4, 15.6)
- moved LED1 0.71 mm to (37.0, 15.6)
- moved LED10 0.71 mm to (50.1, 15.6)
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Connections:
- removed net N$2: C6.1, L1.2, U1.13
- net VCC: now also C6.1, U1.13; no longer L1.1
Routing:
- net VCC: track 81.9 -> 204.1 mm, vias 0 -> 8
- net GND: track 130.0 -> 234.5 mm, vias 3 -> 7
- net SW1: track 0.00 -> 67.5 mm, vias 0 -> 2
- net TXD: track 5.78 -> 40.4 mm, vias 0 -> 3
- net RXD: track 5.89 -> 37.2 mm, vias 0 -> 3
- net LED0: track 0.00 -> 30.3 mm
- net LED1: track 0.05 -> 28.3 mm
- net VMOT: track 40.2 -> 64.2 mm
- net N$28: track 0.00 -> 16.3 mm, vias 0 -> 2
- net LED2: track 16.3 -> 28.1 mm
- net N$10: track 9.03 -> 20.6 mm
- net LED3: track 16.3 -> 26.6 mm
- net LED4: track 17.1 -> 26.5 mm
- net LED5: track 17.2 -> 25.2 mm
- net LED6: track 17.1 -> 23.9 mm
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
Commit message: done
Parts:
- moved R2 0.16 mm to (80.1, 17.3)
Routing:
- net GND: track 234.5 -> 299.8 mm, vias 7 -> 11
- net VCC: track 204.1 -> 257.0 mm, vias 8 -> 9
- net SW1: track 67.5 -> 69.1 mm
- added copper zone on layer 1, net GND
- added copper zone on layer 16, net GND
Other:
- board text added: "bionik_lf"

Commit message: part_values
Parts:
- Q1: value (none) -> 8MHz
- R1: value (none) -> 1M
Changed lines of the file:
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@@
 <?xml version="1.0" encoding="utf-8"?>
 <!DOCTYPE eagle SYSTEM "eagle.dtd">
-<eagle version="8.1.1">
+<eagle version="7.7.0">
 <drawing>
 <settings>
@@
 <setting verticaltext="up"/>
 </settings>
-<grid distance="0.5" unitdist="mm" unit="mm" style="lines" multiple="1" display="no" altdistance="0.025" altunitdist="inch" altunit="inch"/>
+<grid distance="0.1" unitdist="inch" unit="inch" style="lines" multiple="1" display="yes" altdistance="0.025" altunitdist="inch" altunit="inch"/>
 <layers>
 <layer number="1" name="Top" color="4" fill="1" visible="yes" active="yes"/>
@@
 <element name="U$4" library="headers(2mm)" package="1X6" value="1X6" x="25.917040625" y="13.479" rot="R270"/>
 <element name="U$5" library="headers(2mm)" package="1X6" value="1X6" x="114.0310125" y="13.52235" rot="R90"/>
-<element name="Q1" library="crystal-geyer_V1_0" package="3.2X2.5_KX-7" value="" x="81.275671875" y="27.146103125"/>
-<element name="R1" library="rcl" package="R0603" value="" x="81.30469375" y="24.465153125"/>
+<element name="Q1" library="crystal-geyer_V1_0" package="3.2X2.5_KX-7" value="8MHz" x="81.275671875" y="27.146103125"/>
+<element name="R1" library="rcl" package="R0603" value="1M" x="81.30469375" y="24.465153125"/>
 <element name="R2" library="rcl" package="R0603" value="10k" x="80.131003125" y="17.31816875" rot="R90"/>
 <element name="R3" library="rcl" package="R0603" value="10k" x="78.253721875" y="23.655809375" rot="R90"/>

Commit message: cubemx
Parts:
- Q1: value 8MHz -> 16MHz
Changed lines of the file:
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@@
 <element name="U$4" library="headers(2mm)" package="1X6" value="1X6" x="25.917040625" y="13.479" rot="R270"/>
 <element name="U$5" library="headers(2mm)" package="1X6" value="1X6" x="114.0310125" y="13.52235" rot="R90"/>
-<element name="Q1" library="crystal-geyer_V1_0" package="3.2X2.5_KX-7" value="8MHz" x="81.275671875" y="27.146103125"/>
+<element name="Q1" library="crystal-geyer_V1_0" package="3.2X2.5_KX-7" value="16MHz" x="81.275671875" y="27.146103125"/>
 <element name="R1" library="rcl" package="R0603" value="1M" x="81.30469375" y="24.465153125"/>
 <element name="R2" library="rcl" package="R0603" value="10k" x="80.131003125" y="17.31816875" rot="R90"/>
